File: pcb/col2/col2.kicad_pcb (KiCad board)
At the start: 2 copper layers, 48.4 x 17.6 mm, 7 parts

Commit message: adjusted  col unit pcb
Parts:
- D-1-0, D-1-1: footprint custom:Diode_TH_SMD_REVERSIBLE -> crustrusk:Diode_TH_SMD_REVERSIBLE
- SW-1-0, SW-1-1: footprint custom:Kailh_socket_MX -> crustrusk:Kailh_socket_MX
Changed lines of the file:
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@@
 		(property ki_fp_filters "Connector*:*_1x??_*")
 		(sheetname "/")
-		(sheetfile "crustrusk.kicad_sch")
+		(sheetfile "col2.kicad_sch")
 		(units
 			(unit
@@
 		)
 	)
-	(footprint "custom:Kailh_socket_MX"
+	(footprint "crustrusk:Kailh_socket_MX"
 		(layer "F.Cu")
 		(at 70.549005 49.14 90)
@@
 		)
 		(sheetname "/")
-		(sheetfile "crustrusk.kicad_sch")
+		(sheetfile "col2.kicad_sch")
 		(units
 			(unit
@@
 		(embedded_fonts no)
 	)
-	(footprint "custom:Diode_TH_SMD_REVERSIBLE"
+	(footprint "crustrusk:Diode_TH_SMD_REVERSIBLE"
 		(layer "F.Cu")
 		(at 55.379005 49.18 90)
@@
 		(property ki_fp_filters "TO-???* *_Diode_* *SingleDiode* D_*")
 		(sheetname "/")
-		(sheetfile "crustrusk.kicad_sch")
+		(sheetfile "col2.kicad_sch")
 		(units
 			(unit
@@
 		(embedded_fonts no)
 	)
-	(footprint "custom:Kailh_socket_MX"
+	(footprint "crustrusk:Kailh_socket_MX"
 		(layer "F.Cu")
 		(at 51.549005 49.14 90)
@@
 		)
 		(sheetname "/")
-		(sheetfile "crustrusk.kicad_sch")
+		(sheetfile "col2.kicad_sch")
 		(units
 			(unit
@@
 		(embedded_fonts no)
 	)
-	(footprint "custom:Diode_TH_SMD_REVERSIBLE"
+	(footprint "crustrusk:Diode_TH_SMD_REVERSIBLE"
 		(layer "F.Cu")
 		(at 74.379005 49.18 90)
@@
 		(property ki_fp_filters "TO-???* *_Diode_* *SingleDiode* D_*")
 		(sheetname "/")
-		(sheetfile "crustrusk.kicad_sch")
+		(sheetfile "col2.kicad_sch")
 		(units
 			(unit
@@
 	(gr_line
 		(start 82.75 58.6)
-		(end 34.4 58.599958)
+		(end 34.4 58.6)
 		(stroke
 			(width 0.05)
