File: pcb/col2/col2.kicad_sch (KiCad schematic)
At the start: 5 parts

Commit message: adjusted  col unit pcb
Parts:
- D-1-0, D-1-1: footprint custom:Diode_TH_SMD_REVERSIBLE -> crustrusk:Diode_TH_SMD_REVERSIBLE
- SW-1-0, SW-1-1: footprint custom:Kailh_socket_MX -> crustrusk:Kailh_socket_MX
Changed lines of the file:
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@@
 			)
 		)
-		(property "Footprint" "custom:Kailh_socket_MX"
+		(property "Footprint" "crustrusk:Kailh_socket_MX"
 			(at 44.45 20.32 0)
 			(hide yes)
@@
 		)
 		(instances
-			(project "crustrusk"
+			(project "col2"
 				(path "/9e72c485-61d0-44fa-96a5-46ca12df99d7"
 					(reference "SW-1-0")
@@
 			)
 		)
-		(property "Footprint" "custom:Diode_TH_SMD_REVERSIBLE"
+		(property "Footprint" "crustrusk:Diode_TH_SMD_REVERSIBLE"
 			(at 39.37 29.21 0)
 			(hide yes)
@@
 		)
 		(instances
-			(project "crustrusk"
+			(project "col2"
 				(path "/9e72c485-61d0-44fa-96a5-46ca12df99d7"
 					(reference "D-1-0")
@@
 		)
 		(instances
-			(project "crustrusk"
+			(project "col2"
 				(path "/9e72c485-61d0-44fa-96a5-46ca12df99d7"
 					(reference "C1")
@@
 			)
 		)
-		(property "Footprint" "custom:Kailh_socket_MX"
+		(property "Footprint" "crustrusk:Kailh_socket_MX"
 			(at 44.45 36.83 0)
 			(hide yes)
@@
 		)
 		(instances
-			(project "crustrusk"
+			(project "col2"
 				(path "/9e72c485-61d0-44fa-96a5-46ca12df99d7"
 					(reference "SW-1-1")
@@
 			)
 		)
-		(property "Footprint" "custom:Diode_TH_SMD_REVERSIBLE"
+		(property "Footprint" "crustrusk:Diode_TH_SMD_REVERSIBLE"
 			(at 39.37 45.72 0)
 			(hide yes)
@@
 		)
 		(instances
-			(project "crustrusk"
+			(project "col2"
 				(path "/9e72c485-61d0-44fa-96a5-46ca12df99d7"
 					(reference "D-1-1")
