File: pcb/thumb3-boardloaf/thumb3-boardloaf.kicad_sch (KiCad schematic)
At the start: 7 parts

Commit message: Added thumb cluster units
Parts:
- C0: footprint custom:reversible JST_PH_S6B-PH-K_1x06_P2.00mm_Horizontal -> crustrusk:reversible JST_PH_S6B-PH-K_1x06_P2.00mm_Horizontal
- D-0-0, D-0-1, D-0-2: footprint custom:Diode_TH_SMD_REVERSIBLE -> crustrusk:Diode_TH_SMD_REVERSIBLE
- SW-0-0, SW-0-1, SW-0-2: footprint custom:Kailh_hotswap_only_socket_MX_optional_reversible-MIRROR -> crustrusk:Kailh_hotswap_only_socket_MX_optional_reversible-MIRROR
Changed lines of the file:
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@@
 			)
 		)
-		(property "Footprint" "custom:Diode_TH_SMD_REVERSIBLE"
+		(property "Footprint" "crustrusk:Diode_TH_SMD_REVERSIBLE"
 			(at 44.45 46.99 0)
 			(hide yes)
@@
 		)
 		(instances
-			(project "crustrusk"
+			(project "thumb3-boardloaf"
 				(path "/9e72c485-61d0-44fa-96a5-46ca12df99d7"
 					(reference "D-0-1")
@@
 			)
 		)
-		(property "Footprint" "custom:Diode_TH_SMD_REVERSIBLE"
+		(property "Footprint" "crustrusk:Diode_TH_SMD_REVERSIBLE"
 			(at 44.45 30.48 0)
 			(hide yes)
@@
 		)
 		(instances
-			(project "crustrusk"
+			(project "thumb3-boardloaf"
 				(path "/9e72c485-61d0-44fa-96a5-46ca12df99d7"
 					(reference "D-0-0")
@@
 			)
 		)
-		(property "Footprint" "custom:Kailh_hotswap_only_socket_MX_optional_reversible-MIRROR"
+		(property "Footprint" "crustrusk:Kailh_hotswap_only_socket_MX_optional_reversible-MIRROR"
 			(at 49.53 21.59 0)
 			(hide yes)
@@
 		)
 		(instances
-			(project "crustrusk"
+			(project "thumb3-boardloaf"
 				(path "/9e72c485-61d0-44fa-96a5-46ca12df99d7"
 					(reference "SW-0-0")
@@
 			)
 		)
-		(property "Footprint" "custom:Kailh_hotswap_only_socket_MX_optional_reversible-MIRROR"
+		(property "Footprint" "crustrusk:Kailh_hotswap_only_socket_MX_optional_reversible-MIRROR"
 			(at 49.53 38.1 0)
 			(hide yes)
@@
 		)
 		(instances
-			(project "crustrusk"
+			(project "thumb3-boardloaf"
 				(path "/9e72c485-61d0-44fa-96a5-46ca12df99d7"
 					(reference "SW-0-1")
@@
 			)
 		)
-		(property "Footprint" "custom:reversible JST_PH_S6B-PH-K_1x06_P2.00mm_Horizontal"
+		(property "Footprint" "crustrusk:reversible JST_PH_S6B-PH-K_1x06_P2.00mm_Horizontal"
 			(at 25.4 72.39 0)
 			(hide yes)
@@
 		)
 		(instances
-			(project "crustrusk"
+			(project "thumb3-boardloaf"
 				(path "/9e72c485-61d0-44fa-96a5-46ca12df99d7"
 					(reference "C0")
@@
 			)
 		)
-		(property "Footprint" "custom:Kailh_hotswap_only_socket_MX_optional_reversible-MIRROR"
+		(property "Footprint" "crustrusk:Kailh_hotswap_only_socket_MX_optional_reversible-MIRROR"
 			(at 49.53 54.61 0)
 			(hide yes)
@@
 		)
 		(instances
-			(project "crustrusk"
+			(project "thumb3-boardloaf"
 				(path "/9e72c485-61d0-44fa-96a5-46ca12df99d7"
 					(reference "SW-0-2")
@@
 			)
 		)
-		(property "Footprint" "custom:Diode_TH_SMD_REVERSIBLE"
+		(property "Footprint" "crustrusk:Diode_TH_SMD_REVERSIBLE"
 			(at 44.45 63.5 0)
 			(hide yes)
@@
 		)
 		(instances
-			(project "crustrusk"
+			(project "thumb3-boardloaf"
 				(path "/9e72c485-61d0-44fa-96a5-46ca12df99d7"
 					(reference "D-0-2")
