File: pcb/thumb3-boardloaf/thumb3-boardloaf.kicad_pcb (KiCad board)
At the start: 2 copper layers, 23.8 x 67.5 mm, 7 parts

Commit message: Added thumb cluster units
Parts:
- C0: footprint custom:reversible JST_PH_S6B-PH-K_1x06_P2.00mm_Horizontal -> crustrusk:reversible JST_PH_S6B-PH-K_1x06_P2.00mm_Horizontal
- D-0-0, D-0-1, D-0-2: footprint custom:Diode_TH_SMD_REVERSIBLE -> crustrusk:Diode_TH_SMD_REVERSIBLE
- SW-0-0, SW-0-1, SW-0-2: footprint custom:Kailh_hotswap_only_socket_MX_optional_reversible-MIRROR -> crustrusk:Kailh_hotswap_only_socket_MX_optional_reversible-MIRROR
Routing:
- added copper zone on B.Cu, net (none)
- added copper zone on F.Cu, net (none)
- removed copper zone on B.Cu, net GND
- removed copper zone on F.Cu, net GND
Changed lines of the file:
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@@
 		)
 	)
-	(footprint "custom:Diode_TH_SMD_REVERSIBLE"
+	(footprint "crustrusk:Diode_TH_SMD_REVERSIBLE"
 		(layer "F.Cu")
 		(at 43.449961 88.64 180)
@@
 		)
 		(property "Value" "D"
-			(at 0 -0.313125 0)
+			(at 0 -0.313125 180)
 			(layer "F.Fab")
 			(hide yes)
@@
 		)
 		(property "Datasheet" ""
-			(at 0 0 0)
+			(at 0 0 180)
 			(layer "F.Fab")
 			(hide yes)
@@
 		)
 		(property "Description" "Diode"
-			(at 0 0 0)
+			(at 0 0 180)
 			(layer "F.Fab")
 			(hide yes)
@@
 		(property ki_fp_filters "TO-???* *_Diode_* *SingleDiode* D_*")
 		(sheetname "/")
-		(sheetfile "crustrusk.kicad_sch")
+		(sheetfile "thumb3-boardloaf.kicad_sch")
 		(units
 			(unit
@@
 		)
 		(fp_text user "${REFERENCE}"
-			(at 0 2.12 0)
+			(at 0 2.12 180)
 			(layer "B.SilkS")
 			(effects
@@
 		)
 	)
-	(footprint "custom:reversible JST_PH_S6B-PH-K_1x06_P2.00mm_Horizontal"
+	(footprint "crustrusk:reversible JST_PH_S6B-PH-K_1x06_P2.00mm_Horizontal"
 		(layer "F.Cu")
 		(at 53.574961 43.83 180)
@@
 		(tags "connector JST PH horizontal")
 		(property "Reference" "C0"
-			(at 5 -2.55 0)
+			(at 5 -2.55 180)
 			(layer "F.SilkS")
 			(effects
@@
 		)
 		(property "Value" "Conn_01x06_Socket"
-			(at 5 7.45 0)
+			(at 5 7.45 180)
 			(layer "F.Fab")
 			(effects
@@
 		)
 		(property "Datasheet" ""
-			(at 0 0 0)
+			(at 0 0 180)
 			(layer "F.Fab")
 			(hide yes)
@@
 		)
 		(property "Description" "Generic connector, single row, 01x06, script generated"
-			(at 0 0 0)
+			(at 0 0 180)
 			(layer "F.Fab")
 			(hide yes)
@@
 		)
 		(property "KiLib_Generator" "connector/JST"
-			(at 0 0 0)
+			(at 0 0 180)
 			(layer "F.SilkS")
 			(hide yes)
@@
 		(property ki_fp_filters "Connector*:*_1x??_*")
 		(sheetname "/")
-		(sheetfile "crustrusk.kicad_sch")
+		(sheetfile "thumb3-boardloaf.kicad_sch")
 		(units
 			(unit
@@
 		)
 		(fp_text user "${REFERENCE}"
-			(at 5 4.68 0)
+			(at 5 4.68 180)
 			(layer "B.Fab")
 			(effects
@@
 		)
 		(fp_text user "${REFERENCE}"
-			(at 5 2.5 0)
+			(at 5 2.5 180)
 			(layer "F.Fab")
 			(effects
@@
 		)
 	)
-	(footprint "custom:Diode_TH_SMD_REVERSIBLE"
+	(footprint "crustrusk:Diode_TH_SMD_REVERSIBLE"
 		(layer "F.Cu")
 		(at 45.489959 69.54 180)
@@
 		)
 		(property "Value" "D"
-			(at 0 -0.313125 0)
+			(at 0 -0.313125 180)
 			(layer "F.Fab")
 			(hide yes)
@@
 		)
 		(property "Datasheet" ""
-			(at 0 0 0)
+			(at 0 0 180)
 			(layer "F.Fab")
 			(hide yes)
@@
 		)
 		(property "Description" "Diode"
-			(at 0 0 0)
+			(at 0 0 180)
 			(layer "F.Fab")
 			(hide yes)
@@
 		(property ki_fp_filters "TO-???* *_Diode_* *SingleDiode* D_*")
 		(sheetname "/")
-		(sheetfile "crustrusk.kicad_sch")
+		(sheetfile "thumb3-boardloaf.kicad_sch")
 		(units
 			(unit
@@
 		)
 		(fp_text user "${REFERENCE}"
-			(at 0 2.12 0)
+			(at 0 2.12 180)
 			(layer "B.SilkS")
 			(effects
@@
 		)
 	)
-	(footprint "custom:Diode_TH_SMD_REVERSIBLE"
+	(footprint "crustrusk:Diode_TH_SMD_REVERSIBLE"
 		(layer "F.Cu")
 		(at 48.599961 50.49 180)
@@
 		)
 		(property "Value" "D"
-			(at 0 -0.313125 0)
+			(at 0 -0.313125 180)
 			(layer "F.Fab")
 			(hide yes)
@@
 		)
 		(property "Datasheet" ""
-			(at 0 0 0)
+			(at 0 0 180)
 			(layer "F.Fab")
 			(hide yes)
@@
 		)
 		(property "Description" "Diode"
-			(at 0 0 0)
+			(at 0 0 180)
 			(layer "F.Fab")
 			(hide yes)
@@
 		(property ki_fp_filters "TO-???* *_Diode_* *SingleDiode* D_*")
 		(sheetname "/")
-		(sheetfile "crustrusk.kicad_sch")
+		(sheetfile "thumb3-boardloaf.kicad_sch")
 		(units
 			(unit
@@
 		)
 		(fp_text user "${REFERENCE}"
-			(at 0 2.12 0)
+			(at 0 2.12 180)
 			(layer "B.SilkS")
 			(effects
@@
 		)
 	)
-	(footprint "custom:Kailh_hotswap_only_socket_MX_optional_reversible-MIRROR"
+	(footprint "crustrusk:Kailh_hotswap_only_socket_MX_optional_reversible-MIRROR"
 		(layer "F.Cu")
 		(at 45.509961 73.35 180)
@@
 		)
 		(sheetname "/")
-		(sheetfile "crustrusk.kicad_sch")
+		(sheetfile "thumb3-boardloaf.kicad_sch")
 		(units
 			(unit
@@
 		(embedded_fonts no)
 	)
-	(footprint "custom:Kailh_hotswap_only_socket_MX_optional_reversible-MIRROR"
+	(footprint "crustrusk:Kailh_hotswap_only_socket_MX_optional_reversible-MIRROR"
 		(layer "F.Cu")
 		(at 48.509961 54.35 180)
@@
 		)
 		(sheetname "/")
-		(sheetfile "crustrusk.kicad_sch")
+		(sheetfile "thumb3-boardloaf.kicad_sch")
 		(units
 			(unit
@@
 		(embedded_fonts no)
 	)
-	(footprint "custom:Kailh_hotswap_only_socket_MX_optional_reversible-MIRROR"
+	(footprint "crustrusk:Kailh_hotswap_only_socket_MX_optional_reversible-MIRROR"
 		(layer "F.Cu")
 		(at 43.509961 92.35 180)
@@
 		)
 		(sheetname "/")
-		(sheetfile "crustrusk.kicad_sch")
+		(sheetfile "thumb3-boardloaf.kicad_sch")
 		(units
 			(unit
@@
 	)
 	(zone
-		(net "GND")
 		(layers "F.Cu" "B.Cu")
 		(hatch edge 0.5)

Commit message: Added label to thumb clusters
Routing:
- removed copper zone on B.Cu, net (none)
- removed copper zone on F.Cu, net (none)
Other:
- board text added: "Boardloaf"
Changed lines of the file:
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@@
 		(layer "Edge.Cuts")
+	)
+	(gr_text "Boardloaf"
+		(at 37.05 70.45 90)
+		(layer "F.SilkS")
+		(effects
+			(font
+				(size 1 1)
+				(thickness 0.1)
+			)
+		)
+	)
+	(gr_text "Boardloaf"
+		(at 37.05 70.45 90)
+		(layer "B.SilkS")
+		(effects
+			(font
+				(size 1 1)
+				(thickness 0.1)
+			)
+			(justify mirror)
+		)
 	)
 	(segment
@@
 		(net "Net-(D-0-2-A)")
 	)
-	(zone
-		(layers "F.Cu" "B.Cu")
-		(hatch edge 0.5)
-		(connect_pads
-			(clearance 0.5)
-		)
-		(min_thickness 0.25)
-		(fill yes
-			(thermal_gap 0.5)
-			(thermal_bridge_width 0.5)
-			(island_removal_mode 0)
-		)
-		(polygon
-			(pts
-				(xy 28.75 31.84) (xy 143.58 32.26) (xy 143.16 144.16) (xy 28.33 145.62)
-			)
-		)
-	)
 	(embedded_fonts no)
