File: pcb/thumb2-sweep/thumb2-sweep.kicad_pcb (KiCad board)
At the start: 2 copper layers, 55.7 x 38 mm, 5 parts

Commit message: Added label to thumb clusters
Other:
- board text added: "Sweep"
Changed lines of the file:
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@@
 		(fp_poly
 			(pts
-				(xy -3.198439 -0.800549) (xy -2.635868 -0.80055) (xy -2.635868 0.799699) (xy -3.198439 0.799699)
+				(xy -3.19844 -0.800549) (xy -2.635868 -0.80055) (xy -2.635868 0.799699) (xy -3.198439 0.799699)
 			)
 			(stroke
@@
 		(fp_line
 			(start 0.500002 4.18)
-			(end 0.500009 8.539994)
+			(end 0.500008 8.539994)
 			(stroke
 				(width 0.12)
@@
 		)
 		(pad "6" thru_hole oval
-			(at 0 2.180001 60)
+			(at -0.000001 2.180001 60)
 			(size 1.2 1.75)
 			(drill 0.75)
@@
 		(layer "Edge.Cuts")
 	)
+	(gr_text "Sweep"
+		(at 76.8 96.75 355)
+		(layer "F.SilkS")
+		(effects
+			(font
+				(size 1 1)
+				(thickness 0.1)
+			)
+		)
+	)
+	(gr_text "Sweep"
+		(at 76.8 96.75 355)
+		(layer "B.SilkS")
+		(effects
+			(font
+				(size 1 1)
+				(thickness 0.1)
+			)
+			(justify mirror)
+		)
+	)
 	(gr_text "SW_Push"
 		(at 91.102566 112.908882 240)
@@
 	)
 	(segment
-		(start 93.7 113.3)
-		(end 94.432052 116.032045)
-		(width 0.2)
-		(layer "B.Cu")
-		(net "ROW2-0")
-	)
-	(segment
 		(start 91.558681 110.090416)
 		(end 86.744097 114.905)
@@
 	)
 	(segment
-		(start 91.861038 117.925174)
-		(end 93.530553 118.889072)
-		(width 0.2)
-		(layer "F.Cu")
-		(net "ROW0-0")
-	)
-	(segment
-		(start 96.849633 114.194678)
-		(end 96.419551 112.589595)
-		(width 0.2)
-		(layer "F.Cu")
-		(net "ROW0-0")
-	)
-	(segment
-		(start 93.530553 118.889072)
-		(end 94.25073 118.696103)
-		(width 0.2)
-		(layer "F.Cu")
-		(net "ROW0-0")
-	)
-	(segment
-		(start 91.53162 116.695747)
-		(end 91.861038 117.925174)
-		(width 0.2)
-		(layer "F.Cu")
-		(net "ROW0-0")
-	)
-	(segment
-		(start 94.25073 118.696103)
-		(end 96.849633 114.194678)
-		(width 0.2)
-		(layer "F.Cu")
-		(net "ROW0-0")
-	)
-	(segment
-		(start 70.080177 105.180177)
-		(end 81.595744 116.695744)
-		(width 0.2)
-		(layer "B.Cu")
-		(net "ROW0-0")
-	)
-	(segment
-		(start 81.595744 116.695744)
-		(end 91.531611 116.695744)
-		(width 0.2)
-		(layer "B.Cu")
-		(net "ROW0-0")
-	)
-	(segment
-		(start 68.213899 105.180177)
-		(end 70.080177 105.180177)
-		(width 0.2)
-		(layer "B.Cu")
-		(net "ROW0-0")
-	)
-	(segment
 		(start 63.566749 92.334321)
 		(end 64.700599 92.334321)
@@
 	)
 	(segment
+		(start 91.861038 117.925174)
+		(end 93.530553 118.889072)
+		(width 0.2)
+		(layer "F.Cu")
+		(net "ROW0-0")
+	)
+	(segment
+		(start 96.849633 114.194678)
+		(end 96.419551 112.589595)
+		(width 0.2)
+		(layer "F.Cu")
+		(net "ROW0-0")
+	)
+	(segment
+		(start 93.530553 118.889072)
+		(end 94.25073 118.696103)
+		(width 0.2)
+		(layer "F.Cu")
+		(net "ROW0-0")
+	)
+	(segment
+		(start 91.53162 116.695747)
+		(end 91.861038 117.925174)
+		(width 0.2)
+		(layer "F.Cu")
+		(net "ROW0-0")
+	)
+	(segment
+		(start 94.25073 118.696103)
+		(end 96.849633 114.194678)
+		(width 0.2)
+		(layer "F.Cu")
+		(net "ROW0-0")
+	)
+	(segment
+		(start 70.080177 105.180177)
+		(end 81.595744 116.695744)
+		(width 0.2)
+		(layer "B.Cu")
+		(net "ROW0-0")
+	)
+	(segment
+		(start 81.595744 116.695744)
+		(end 91.531611 116.695744)
+		(width 0.2)
+		(layer "B.Cu")
+		(net "ROW0-0")
+	)
+	(segment
+		(start 68.213899 105.180177)
+		(end 70.080177 105.180177)
+		(width 0.2)
+		(layer "B.Cu")
+		(net "ROW0-0")
+	)
+	(segment
+		(start 93.7 113.3)
+		(end 94.432052 116.032045)
+		(width 0.2)
+		(layer "B.Cu")
+		(net "ROW2-0")
+	)
+	(segment
