File: pcb/thumb3-cheapino/thumb3-cheapino.kicad_pcb (KiCad board)
At the start: 2 copper layers, 72.6 x 33 mm, 7 parts

Commit message: Added label to thumb clusters
Other:
- board text added: "Cheapino"
Changed lines of the file:
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@@
 			(pts
 				(xy 3.19853 -0.800292) (xy -3.201338 -0.800292) (xy -3.201338 -0.651431) (xy -3.053026 -0.651431)
-				(xy 3.050219 -0.651431) (xy 3.050219 0.649231) (xy -3.053026 0.649232) (xy -3.053026 -0.651431)
-				(xy -3.201338 -0.651431) (xy -3.201338 0.800708) (xy 3.198529 0.800709)
+				(xy 3.050219 -0.651431) (xy 3.05022 0.649231) (xy -3.053026 0.649232) (xy -3.053026 -0.651431) (xy -3.201338 -0.651431)
+				(xy -3.201338 0.800708) (xy 3.198528 0.800709)
 			)
 			(stroke
@@
 		(fp_poly
 			(pts
-				(xy 3.198529 0.800292) (xy -3.201338 0.800292) (xy -3.201338 0.651431) (xy -3.053026 0.651431) (xy 3.050219 0.651431)
+				(xy 3.198529 0.800291) (xy -3.201338 0.800292) (xy -3.201338 0.651431) (xy -3.053026 0.651431) (xy 3.050219 0.651431)
 				(xy 3.050219 -0.649231) (xy -3.053026 -0.649232) (xy -3.053026 0.651431) (xy -3.201338 0.651431)
 				(xy -3.201339 -0.800709) (xy 3.198529 -0.800709)
@@
 		)
 		(pad "1" thru_hole rect
-			(at -3.810001 0 350)
+			(at -3.810002 0 350)
 			(size 1.397 1.397)
 			(drill 0.8128)
@@
 		)
 		(pad "2" thru_hole circle
-			(at 3.810001 0 350)
+			(at 3.810002 0 350)
 			(size 1.397 1.397)
 			(drill 0.8128)
@@
 		)
 		(fp_line
-			(start 12.059996 -1.459996)
+			(start 12.059996 -1.459997)
 			(end 11.140003 -1.460004)
 			(stroke
@@
 		(fp_line
 			(start 12.06 6.360004)
-			(end 12.059996 -1.459996)
+			(end 12.059996 -1.459997)
 			(stroke
 				(width 0.12)
@@
 		(fp_poly
 			(pts
-				(xy -1.299998 2.499997) (xy -0.29999 2.50001) (xy -0.3 4.099999) (xy -1.299998 4.100006)
+				(xy -1.299998 2.499997) (xy -0.29999 2.50001) (xy -0.3 4.099999) (xy -1.299997 4.100006)
 			)
 			(stroke
@@
 		(fp_poly
 			(pts
-				(xy 10.299996 4.680007) (xy 11.299998 4.679993) (xy 11.299994 6.280004) (xy 10.300005 6.279997)
+				(xy 10.299996 4.680007) (xy 11.299998 4.679993) (xy 11.299994 6.280005) (xy 10.300005 6.279997)
 			)
 			(stroke
@@
 		(layer "Edge.Cuts")
 	)
+	(gr_text "Cheapino"
+		(at 59.55 57.55 0)
+		(layer "F.SilkS")
+		(effects
+			(font
+				(size 1 1)
+				(thickness 0.1)
+			)
+		)
+	)
+	(gr_text "Cheapino"
+		(at 59.55 57.55 0)
+		(layer "B.SilkS")
+		(effects
+			(font
+				(size 1 1)
+				(thickness 0.1)
+			)
+			(justify mirror)
+		)
+	)
 	(gr_text "SW_Push"
 		(at 97.544488 75.967115 247)
@@
 	)
 	(segment
-		(start 56.035 61.754292)
-		(end 54.765 60.484292)
+		(start 84.542877 75.761314)
+		(end 99.764645 75.761314)
+		(width 0.2)
+		(layer "B.Cu")
+		(net "ROW2-0")
+	)
+	(segment
+		(start 99.764645 75.761314)
+		(end 99.994775 75.991444)
+		(width 0.2)
+		(layer "B.Cu")
+		(net "ROW2-0")
+	)
+	(segment
+		(start 100.170226 76.038771)
+		(end 101.229774 78.661236)
+		(width 0.2)
+		(layer "B.Cu")
+		(net "ROW2-0")
+	)
+	(segment
+		(start 97.701474 73.165845)
+		(end 97.701474 70.508118)
 		(width 0.2)
 		(layer "F.Cu")
-		(net "Net-(D-0-0-A)")
+		(net "Net-(D-0-2-A)")
 	)
 	(segment
-		(start 56.035 66.875)
-		(end 52.31 70.6)
+		(start 97.701474 73.165845)
+		(end 92.128633 78.738686)
 		(width 0.2)
 		(layer "F.Cu")
-		(net "Net-(D-0-0-A)")
+		(net "Net-(D-0-2-A)")
 	)
 	(segment
-		(start 56.035 63.024292)
-		(end 56.035 66.875)
+		(start 97.701474 70.508118)
+		(end 97.52489 70.331534)
 		(width 0.2)
 		(layer "F.Cu")
-		(net "Net-(D-0-0-A)")
+		(net "Net-(D-0-2-A)")
 	)
 	(segment
-		(start 56.035 63.024292)
-		(end 56.035 61.754292)
+		(start 92.128633 78.738686)
+		(end 91.557123 78.738686)
 		(width 0.2)
 		(layer "F.Cu")
-		(net "Net-(D-0-0-A)")
+		(net "Net-(D-0-2-A)")
 	)
 	(via
-		(at 54.765 60.484292)
+		(at 97.52489 70.331534)
 		(size 0.6)
 		(drill 0.3)
 		(layers "F.Cu" "B.Cu")
-		(net "Net-(D-0-0-A)")
+		(net "Net-(D-0-2-A)")
+	)
+	(segment
+		(start 77.486574 66.986477)
+		(end 77.486574 65.795661)
+		(width 0.2)
+		(layer "F.Cu")
+		(net "Net-(D-0-1-A)")
+	)
+	(segment
+		(start 72.552118 72.9616)
+		(end 72.552118 71.920933)
+		(width 0.2)
+		(layer "F.Cu")
+		(net "Net-(D-0-1-A)")
+	)
+	(segment
+		(start 77.486574 65.795661)
+		(end 77.486574 63.883355)
+		(width 0.2)
+		(layer "F.Cu")
+		(net "Net-(D-0-1-A)")
+	)
+	(segment
+		(start 72.552118 71.920933)
+		(end 77.486574 66.986477)
+		(width 0.2)
+		(layer "F.Cu")
+		(net "Net-(D-0-1-A)")
+	)
+	(segment
+		(start 77.486574 63.883355)
+		(end 76.676935 63.073716)
+		(width 0.2)
+		(layer "F.Cu")
+		(net "Net-(D-0-1-A)")
+	)
+	(via
+		(at 76.676935 63.073716)
+		(size 0.6)
+		(drill 0.3)
+		(layers "F.Cu" "B.Cu")
+		(net "Net-(D-0-1-A)")
 	)
 	(segment
@@
 	)
 	(segment
-		(start 97.701474 73.165845)
-		(end 97.701474 70.508118)
+		(start 56.035 61.754292)
+		(end 54.765 60.484292)
 		(width 0.2)
 		(layer "F.Cu")
-		(net "Net-(D-0-2-A)")
+		(net "Net-(D-0-0-A)")
 	)
 	(segment
-		(start 97.701474 73.165845)
-		(end 92.128633 78.738686)
+		(start 56.035 66.875)
+		(end 52.31 70.6)
 		(width 0.2)
 		(layer "F.Cu")
-		(net "Net-(D-0-2-A)")
+		(net "Net-(D-0-0-A)")
 	)
 	(segment
-		(start 97.701474 70.508118)
-		(end 97.52489 70.331534)
+		(start 56.035 63.024292)
+		(end 56.035 66.875)
 		(width 0.2)
 		(layer "F.Cu")
-		(net "Net-(D-0-2-A)")
+		(net "Net-(D-0-0-A)")
 	)
 	(segment
-		(start 92.128633 78.738686)
-		(end 91.557123 78.738686)
+		(start 56.035 63.024292)
+		(end 56.035 61.754292)
 		(width 0.2)
 		(layer "F.Cu")
-		(net "Net-(D-0-2-A)")
+		(net "Net-(D-0-0-A)")
 	)
 	(via
-		(at 97.52489 70.331534)
+		(at 54.765 60.484292)
 		(size 0.6)
 		(drill 0.3)
 		(layers "F.Cu" "B.Cu")
-		(net "Net-(D-0-2-A)")
+		(net "Net-(D-0-0-A)")
 	)
 	(segment
@@
 	)
 	(segment
-		(start 77.486574 66.986477)
-		(end 77.486574 65.795661)
-		(width 0.2)
-		(layer "F.Cu")
-		(net "Net-(D-0-1-A)")
-	)
-	(segment
-		(start 72.552118 72.9616)
-		(end 72.552118 71.920933)
-		(width 0.2)
-		(layer "F.Cu")
-		(net "Net-(D-0-1-A)")
-	)
-	(segment
-		(start 77.486574 65.795661)
-		(end 77.486574 63.883355)
-		(width 0.2)
-		(layer "F.Cu")
-		(net "Net-(D-0-1-A)")
-	)
-	(segment
-		(start 72.552118 71.920933)
-		(end 77.486574 66.986477)
-		(width 0.2)
-		(layer "F.Cu")
-		(net "Net-(D-0-1-A)")
-	)
-	(segment
-		(start 77.486574 63.883355)
-		(end 76.676935 63.073716)
-		(width 0.2)
-		(layer "F.Cu")
-		(net "Net-(D-0-1-A)")
-	)
-	(via
-		(at 76.676935 63.073716)
-		(size 0.6)
-		(drill 0.3)
-		(layers "F.Cu" "B.Cu")
-		(net "Net-(D-0-1-A)")
-	)
-	(segment
-		(start 84.542877 75.761314)
-		(end 99.764645 75.761314)
-		(width 0.2)
-		(layer "B.Cu")
-		(net "ROW2-0")
-	)
-	(segment
-		(start 99.764645 75.761314)
-		(end 99.994775 75.991444)
-		(width 0.2)
-		(layer "B.Cu")
-		(net "ROW2-0")
-	)
-	(segment
-		(start 100.170226 76.038771)
-		(end 101.229774 78.661236)
-		(width 0.2)
-		(layer "B.Cu")
-		(net "ROW2-0")
-	)
-	(segment
