File: pcb/thumb3-corne/thumb3-corne.kicad_pcb (KiCad board)
At the start: 2 copper layers, 74.1 x 30.4 mm, 7 parts

Commit message: Added label to thumb clusters
Other:
- board text added: "Corne"
Changed lines of the file:
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@@
 		(fp_poly
 			(pts
-				(xy 3.19853 -0.800291) (xy -3.201338 -0.800292) (xy -3.201337 -0.651431) (xy -3.053026 -0.651431)
+				(xy 3.19853 -0.800291) (xy -3.201338 -0.800292) (xy -3.201337 -0.65143) (xy -3.053026 -0.651431)
 				(xy 3.050219 -0.651432) (xy 3.050219 0.649232) (xy -3.053026 0.649232) (xy -3.053026 -0.651431)
-				(xy -3.201337 -0.651431) (xy -3.201339 0.800709) (xy 3.19853 0.800709)
+				(xy -3.201337 -0.65143) (xy -3.201339 0.800709) (xy 3.19853 0.800709)
 			)
 			(stroke
@@
 		(fp_poly
 			(pts
-				(xy -2.635868 0.80055) (xy -3.198439 0.80055) (xy -3.198439 -0.799699) (xy -2.635868 -0.799699)
+				(xy -2.635868 0.80055) (xy -3.198439 0.80055) (xy -3.198439 -0.799699) (xy -2.635868 -0.7997)
 			)
 			(stroke
@@
 		)
 		(pad "1" smd rect
-			(at -2.75 0.000001 66.12)
+			(at -2.750001 0.000001 66.12)
 			(size 2 0.5)
 			(layers "F.Cu")
@@
 		)
 		(pad "1" smd rect
-			(at -2.75 0.000001 246.12)
+			(at -2.750001 0.000001 246.12)
 			(size 2 0.5)
 			(layers "B.Cu")
@@
 		)
 		(pad "2" smd rect
-			(at 2.75 -0.000001 66.12)
+			(at 2.750001 -0.000001 66.12)
 			(size 2 0.5)
 			(layers "F.Cu")
@@
 		)
 		(pad "2" smd rect
-			(at 2.75 -0.000001 246.12)
+			(at 2.750001 -0.000001 246.12)
 			(size 2 0.5)
 			(layers "B.Cu")
@@
 			)
 		)
-		(fp_text user "1.00u"
-			(at -5.715001 -8.255 0)
-			(layer "Dwgs.User")
-			(effects
-				(font
-					(size 1.524 1.524)
-					(thickness 0.3048)
-				)
-			)
-		)
 		(fp_text user "${REFERENCE}"
 			(at 0.635 4.445 0)
@@
 		)
 		(fp_line
-			(start 5.080001 6.985002)
+			(start 5.080001 6.985003)
 			(end -3.809999 6.985001)
 			(stroke
@@
 		(fp_line
 			(start 5.08 6.604001)
-			(end 5.080001 6.985002)
+			(end 5.080001 6.985003)
 			(stroke
 				(width 0.15)
@@
 		)
 		(fp_line
-			(start 5.080001 6.985002)
+			(start 5.080001 6.985003)
 			(end -3.809999 6.985001)
 			(stroke
@@
 		(fp_line
 			(start 5.079997 2.54)
-			(end 5.080001 6.985002)
+			(end 5.080001 6.985003)
 			(stroke
 				(width 0.12)
@@
 					(size 1 1)
 					(thickness 0.15)
-				)
-			)
-		)
-		(fp_text user "1.00u"
-			(at -5.715 -8.255 168.06)
-			(layer "Dwgs.User")
-			(effects
-				(font
-					(size 1.524 1.524)
-					(thickness 0.3048)
 				)
 			)
@@
 			)
 		)
-		(fp_text user "1.00u"
-			(at -5.715001 -8.255 66.12)
-			(layer "Dwgs.User")
-			(effects
-				(font
-					(size 1.524 1.524)
-					(thickness 0.3048)
-				)
-			)
-		)
 		(fp_text user "${REFERENCE}"
 			(at 0.635 4.445 66.12)
@@
 		(layer "Edge.Cuts")
 	)
+	(gr_text "Corne"
+		(at 73 36.95 0)
+		(layer "F.SilkS")
+		(effects
+			(font
+				(size 1 1)
+				(thickness 0.1)
+			)
+		)
+	)
+	(gr_text "Corne"
+		(at 73 36.95 0)
+		(layer "B.SilkS")
+		(effects
+			(font
+				(size 1 1)
+				(thickness 0.1)
+			)
+			(justify mirror)
+		)
+	)
 	(gr_text "SW_Push"
