File: pcb/thumb4-elephant42/thumb4-elephant42.kicad_pcb (KiCad board)
At the start: 2 copper layers, 84.5 x 60 mm, 9 parts

Commit message: Added label to thumb clusters
Other:
- board text added: "Elephant42"
