File: pcb/thumb4-nyx/thumb4-nyx.kicad_pcb (KiCad board)
At the start: 2 copper layers, 64 x 60.7 mm, 9 parts

Commit message: Updated Nyx thumb slightly
Parts:
- moved C0 26.0 mm to (125.7, 133.9)
Routing:
- net ROW2-0: track 9.85 -> 34.7 mm
- net COL0: track 121.1 -> 134.7 mm
- net ROW3-0: track 38.9 -> 26.0 mm
- net ROW0-0: track 58.0 -> 65.0 mm
- net ROW1-0: track 31.5 -> 35.3 mm
Other:
- board size 64 x 60.7 mm -> 70.8 x 53.7 mm

Commit message: Nyx thumb update 2
Parts:
- moved C0 16.2 mm to (133.8, 119.9), turned to 135 degrees
Routing:
- net ROW2-0: track 34.7 -> 49.9 mm
- net ROW1-0: track 35.3 -> 45.7 mm
- net COL0: track 134.7 -> 129.9 mm
- net ROW0-0: track 65.0 -> 66.8 mm
- net ROW3-0: track 26.0 -> 26.8 mm
Other:
- board size 70.8 x 53.7 mm -> 71 x 57.6 mm
